File: BMSv1.1/untitled.brd (EAGLE design)
At the start: 66.1 x 60 mm, 61 parts, among them J1 U.FL-R-SMT(01), J3 10103594, Q1 MMBT3904, Q2 MMBT3904, Q3 12MHz, U3 PCF8574AT, U4 ADS1115IDGSR, U5 AMS1117, U6 AMS1117

Commit message: fix PCB v1.0
Parts:
- C11, C19, C5, C7, C9: value 10uF -> 1uF
- R12, R13, R3: value 1K -> 330
- R4, R5: value 1K -> 10K
Routing:
- net 3V3: track 163.4 -> 164.7 mm
