File: BMSv1.2/untitled.sch (EAGLE design)
At the start: 61 parts, among them J1 U.FL-R-SMT(01), J3 10103594, Q1 MMBT3904, Q2 MMBT3904, Q3 12MHz, U3 PCF8574AT, U4 ADS1115IDGSR, U5 AMS1117, U6 AMS1117

Commit message: PCB BMS v1.2
Parts:
- removed C4: 100nF, rcl:C-EUC0805K
- removed CONN3.2: (no value), CONN3.5:CONN3.5
- removed FUSE-KOTAK1: (no value), FUSE-KOTAK:FUSE-KOTAK
- removed PS2: LD05-23B05R2, LD05-23B05R2:LD05-23B05R2
- removed U3: PCF8574AT, PCF8574AT:PCF8574AT
- removed U4: ADS1115IDGSR, ADS1115IDGSR:ADS1115IDGSR
- removed U5, U6: AMS1117, AMS1117:AMS1117
- added HEADER-3.81-1: (no value), HEADER-3.81-4:HEADER-3.81-4
- added IC1: MCP23017SS, microchip:MCP23017SS
- added R16: 4.7K, adafruit:R-US_M0805
- added TTL-RS2: (no value), TTL-RS485:TTL-RS485
- added U1, U2: RT9193-33GB, RT9193-33GB:RT9193-33GB
- PS1: value URB4805YMD-6WR3 -> URB2405YMD-10WR3; device URB4805YMD-6WR3:URB4805YMD-6WR3 -> URB2405YMD-10WR3:URB2405YMD-10WR3
- R10, R11, R14, R6, R9: value 10K -> 10k
- R15: value (none) -> 10k; device adafruit:R-US_0207/10 -> adafruit:R-US_M0805
Connections:
- removed net A+: CONN2P-3.5PI3.P1, TTL-RS1.A
- removed net ADS0: U4.AIN0
- removed net ADS1: U4.AIN1
- removed net ADS2: U4.AIN2
- removed net ADS3: U4.AIN3
- removed net B-: CONN2P-3.5PI3.P0, TTL-RS1.B
- removed net DO0: CONN3.2.P4, U3.P0
- removed net DO1: CONN3.2.P3, U3.P1
- removed net DO2: CONN3.2.P2, U3.P2
- removed net DO3: CONN3.2.P1, U3.P3
- removed net RX_RS485: MD1.IO16, TTL-RS1.RX
- removed net TX_RS485: MD1.IO17, TTL-RS1.TX
- new net N$11: CONN2P-3.5PI1.P0, PS1.CTRL, PS1.VIN
- new net N$17: CONN3.1.P2, IC1.GPA1
- new net N$18: IC1.A0, R11.1
- new net N$19: IC1.A1, R14.1
- new net N$20: IC1.A2, R15.1
- new net N$21: CONN3.1.P3, IC1.GPA2
- new net N$22: CONN3.1.P4, IC1.GPA3
- new net RX-PZEM: MD1.IO15, TTL-RS2.RX
- new net RX-RS485: MD1.IO17, TTL-RS1.RX
- new net TX-PZEM: MD1.IO14, TTL-RS2.TX
- new net TX-RS485: MD1.IO16, TTL-RS1.TX
- net 1WIRE: now also CONN3.1.P5, CONN3.1.P6, CONN3.1.P7, CONN3.1.P8, MD1.IO4, R16.2; no longer CONN3.2.P5, CONN3.2.P6, CONN3.2.P7, CONN3.2.P8, MD1.IO14, R15.1
- net 3V3: now also HEADER-3.81-1.3, HEADER-3.81-1.4, R16.1, U1.VOUT; no longer CONN3.1.P1, CONN3.1.P2, R15.2, U5.VOUT
- net 3V3-LORA-RS232: now also U2.VOUT; no longer C4.1, R6.2, R9.1, U3.VDD, U4.VDD, U6.VOUT
- net GND: now also CONN2P-3.5PI1.P1, HEADER-3.81-1.1, HEADER-3.81-1.2, IC1.VSS, PS1.GND, R11.2, R14.2, R15.2, TTL-RS2.GND, U1.GND, U2.GND; no longer C4.2, CONN3.1.P3, CONN3.1.P4, CONN3.1.P5, PS2.-VO, R10.1, R11.1, R14.1, U3.VSS, U4.ADDR, U4.GND, U5.ADJ/GND, U6.ADJ/GND
- net LED_WARNING: now also MD1.IO33; no longer MD1.IO15
- net LORA_DI0: now also MD1.IO32; no longer MD1.IO25
- net LORA_DI1: now also MD1.IO25; no longer MD1.IO32
- net N$10: now also CONN2P-3.5PI2.P0, TTL-RS1.B; no longer R14.2, U3.A0
- net N$13: now also CONN2P-3.5PI3.P0, TTL-RS2.B; no longer FUSE-KOTAK1.2, PS1.VIN, PS2.AC(L)
- net N$14: now also IC1.!RESET, R6.1; no longer R11.2, U3.A1
- net N$15: now also CONN3.1.P1, IC1.GPA0; no longer R10.2, U3.A2
- net N$16: no longer PS2.+VO
- net N$6: now also CONN2P-3.5PI3.P1, TTL-RS2.A; no longer CONN2P-3.5PI1.P0, PS1.GND, PS2.AC(N)
- net N$7: now also CONN2P-3.5PI2.P1, TTL-RS1.A; no longer CONN2P-3.5PI1.P1, FUSE-KOTAK1.1
- net OUT+: now also IC1.VDD, R10.2, R6.2, R9.2, TTL-RS2.VCC, U1.EN, U1.VIN, U2.EN, U2.VIN; no longer CONN3.1.P6, CONN3.1.P7, CONN3.1.P8, U5.VIN, U6.VIN
- net SCL: now also IC1.SCL, R9.1; no longer CONN2P-3.5PI2.P1, R9.2, U3.SCL, U4.SCL
- net SDA: now also IC1.SDA, R10.1; no longer CONN2P-3.5PI2.P0, R6.1, U3.SDA, U4.SDA
Other:
- note removed: "LED"
- moved on the sheet: D1, D6, POWER, PROSES, R10, R11, R12, R13, R14, R15, R3, R4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
